Commit message: #1 Add Arm control to steering code.

File: rover_22_robotic_arm/arm_22_gazebo_pos/urdf/assembly.urdf.xacro (robot description, xacro)
@@ -1,14 +1,15 @@
 <?xml version="1.0" ?>
 <robot name="assembly" xmlns:xacro="http://www.ros.org/wiki/xacro">
-<xacro:include filename="$(find arm_22_gazebo_pos)/urdf/materials.xacro" />
+<!-- <xacro:include filename="$(find arm_22_gazebo_pos)/urdf/materials.xacro" /> -->
 <xacro:include filename="$(find arm_22_gazebo_pos)/urdf/assembly.trans" />
 <xacro:include filename="$(find arm_22_gazebo_pos)/urdf/assembly.gazebo" />
-<link name="world"> </link>
+<xacro:include filename="$(find rover_22_description)/urdf/rover_22.xacro" />
+<!-- <link name="world"> </link> -->
 <joint name="dummy_joint" type="fixed">
-  <origin xyz="0 0 0.06" rpy="0 0 0"/>
-  <parent link="world"/>
-  <child link="base_link"/>
-</joint>
-<link name="base_link">
+  <origin xyz="0.39 0.3 0.07" rpy="0 0 3.14"/>
+  <parent link="base_link"/>
+  <child link="alt_plaka"/>
+</joint>
+<link name="alt_plaka">
   <inertial>
     <origin rpy="0 0 0" xyz="2.111478230178841e-13 0.011682408428370204 0.005554773279956959"/>
@@ -19,5 +20,5 @@
     <origin rpy="0 0 0" xyz="0 0 0"/>
     <geometry>
-      <mesh filename="package://arm_22_gazebo_pos/meshes/base_link.stl" scale="0.001 0.001 0.001"/>
+      <mesh filename="package://arm_22_gazebo_pos/meshes/alt_plaka.stl" scale="0.001 0.001 0.001"/>
     </geometry>
     <material name="silver"/>
@@ -26,5 +27,5 @@
     <origin rpy="0 0 0" xyz="0 0 0"/>
     <geometry>
-      <mesh filename="package://arm_22_gazebo_pos/meshes/base_link.stl" scale="0.001 0.001 0.001"/>
+      <mesh filename="package://arm_22_gazebo_pos/meshes/alt_plaka.stl" scale="0.001 0.001 0.001"/>
     </geometry>
   </collision>
@@ -192,5 +193,5 @@
 <joint name="axis_1" type="continuous">
   <origin rpy="0 0 0" xyz="0.0 0.0 0.0535"/>
-  <parent link="base_link"/>
+  <parent link="alt_plaka"/>
   <child link="1_2_link_1"/>
   <axis xyz="0.0 0.0 1.0"/>

File: rover_22_robotic_arm/rover_22_description/urdf/rover_22.xacro (robot description, xacro)
@@ -296,5 +296,5 @@
     </plugin>
   </gazebo>
-  <gazebo reference="camera">
+  <!-- <gazebo reference="camera">
     <sensor type="camera" name="camera">
       <update_rate>30.0</update_rate>
@@ -331,4 +331,4 @@
       </plugin>
     </sensor>
-  </gazebo>
+  </gazebo> -->
 </robot>
