Commit message: Thu 13 Jan 23:52:26 +03 2022

File: marsyard/urdf/marsyard_Grid.urdf.xacro (robot description, xacro)
@@ -1,5 +1,6 @@
+<?xml version="1.0" encoding="utf-8"?>
 <robot name="robot">
 <!--
-@author: Baran Berk Bağcı-->
+@author: Baran Berk Bagci-->
 <!-- Marsyard grid urdf this is marsyard surface -->
   <link name="marsyard_Grid_link">

File: rover_22_robotic_arm/rover_22_description/urdf/rover_22.xacro (robot description, xacro)
@@ -18,10 +18,10 @@
       <material name="silver" />
     </visual>
-    <collision>
+    <!-- <collision>
       <origin rpy="0 0 0" xyz="0 0 0" />
       <geometry>
         <mesh filename="package://rover_22_description/meshes/base_link.stl" scale="0.001 0.001 0.001" />
       </geometry>
-    </collision>
+    </collision> -->
   </link>
   <link name="steering_leftfront_link_1">
@@ -38,10 +38,10 @@
       <material name="silver" />
     </visual>
-    <collision>
+    <!-- <collision>
       <origin rpy="0 0 0" xyz="0.071 -0.460515 0.071298" />
       <geometry>
         <mesh filename="package://rover_22_description/meshes/steering_leftfront_link_1.stl" scale="0.001 0.001 0.001" />
       </geometry>
-    </collision>
+    </collision> -->
   </link>
   <link name="steering_leftrear_link_1">
@@ -58,10 +58,10 @@
       <material name="silver" />
     </visual>
-    <collision>
+    <!-- <collision>
       <origin rpy="0 0 0" xyz="0.071 0.460515 0.071298" />
       <geometry>
         <mesh filename="package://rover_22_description/meshes/steering_leftrear_link_1.stl" scale="0.001 0.001 0.001" />
       </geometry>
-    </collision>
+    </collision> -->
   </link>
   <link name="steering_rightrear_link_1">
@@ -78,10 +78,10 @@
       <material name="silver" />
     </visual>
-    <collision>
+    <!-- <collision>
       <origin rpy="0 0 0" xyz="-0.851 0.460515 0.071298" />
       <geometry>
         <mesh filename="package://rover_22_description/meshes/steering_rightrear_link_1.stl" scale="0.001 0.001 0.001" />
       </geometry>
-    </collision>
+    </collision> -->
   </link>
   <link name="steering_rightfront_link_1">
@@ -98,10 +98,10 @@
       <material name="silver" />
     </visual>
-    <collision>
+    <!-- <collision>
       <origin rpy="0 0 0" xyz="-0.851 -0.460515 0.071298" />
       <geometry>
         <mesh filename="package://rover_22_description/meshes/steering_rightfront_link_1.stl" scale="0.001 0.001 0.001" />
       </geometry>
-    </collision>
+    </collision> -->
   </link>
   <link name="wheel_leftfront_link_1">
