Commit message: #5 Final changes.

File: rover_22_descriptions/rover_22_description_velodyne/urdf/rover_22.xacro (robot description, xacro)
@@ -2,5 +2,5 @@
 <robot name="rover_22" xmlns:xacro="http://www.ros.org/wiki/xacro">
   <xacro:include filename="$(find rover_22_description_velodyne)/urdf/vlp16.urdf.xacro" />
-  <xacro:property name="cameraSize" value="0.05" />
+  <xacro:property name="cameraSize" value="0.02" />
   <xacro:property name="cameraMass" value="0.1" />
   <xacro:include filename="$(find rover_22_description_velodyne)/urdf/materials.xacro" />
@@ -237,5 +237,5 @@
   <vlp16 prefix="base" topic="/velodyne_points" hz="10" samples="440" gpu="true" max_range="5.0" min_range="0.1" min_angle="-2.39982772" max_angle="2.39982772" />
   <joint name="base_laser_joint" type="fixed">
-    <origin xyz="0.45 0.30 0.12" rpy="0 0 1.57" />
+    <origin xyz="0.45 -0.1 0.09" rpy="0 0 1.57" />
     <parent link="base_link" />
     <child link="velodyne" />
@@ -265,5 +265,5 @@
   <joint name="camera_joint" type="fixed">
     <axis xyz="1 1 0" />
-    <origin xyz="0.45 0.30 0.22" rpy="0 0 1.57" />
+    <origin xyz="0.45 -0.10 0.19" rpy="0 0 1.57" />
     <parent link="base_link" />
     <child link="camera" />

File: rover_22_robotic_arm/arm_22_gazebo_pos/urdf/_d435.urdf.xacro (robot description, xacro)
@@ -53,10 +53,10 @@
         <material name="${name}_aluminum"/>
       </visual>
-      <collision>
+      <!-- <collision>
         <origin xyz="0 ${-d435_cam_depth_py} 0" rpy="0 0 0"/>
         <geometry>
         <box size="${d435_cam_depth} ${d435_cam_width} ${d435_cam_height}"/>
         </geometry>
-      </collision>
+      </collision> -->
       <inertial>
         <!-- The following are not reliable values, and should not be used for modeling -->

File: rover_22_robotic_arm/arm_22_gazebo_pos/urdf/assembly.urdf.xacro (robot description, xacro)
@@ -1,251 +1,244 @@
 <?xml version="1.0" ?>
-<robot name="assembly" xmlns:xacro="http://www.ros.org/wiki/xacro">
-<!-- <xacro:include filename="$(find arm_22_gazebo_pos)/urdf/materials.xacro" /> -->
-<xacro:include filename="$(find arm_22_gazebo_pos)/urdf/assembly.trans" />
-<xacro:include filename="$(find arm_22_gazebo_pos)/urdf/assembly.gazebo" />
-<xacro:include filename="$(find rover_22_description)/urdf/rover_22.xacro" />
-<!-- <link name="world"> </link> -->
-<joint name="dummy_joint" type="fixed">
-  <origin xyz="0.39 0.3 0.07" rpy="0 0 3.14"/>
-  <parent link="base_link"/>
-  <child link="alt_plaka"/>
-</joint>
-<link name="alt_plaka">
-  <inertial>
-    <origin rpy="0 0 0" xyz="2.111478230178841e-13 0.011682408428370204 0.005554773279956959"/>
-    <mass value="4.192131083267752"/>
-    <inertia ixx="0.007549" ixy="0.0" ixz="0.0" iyy="0.013998" iyz="0.000517" izz="0.018961"/>
-  </inertial>
-  <visual>
-    <origin rpy="0 0 0" xyz="0 0 0"/>
-    <geometry>
-      <mesh filename="package://arm_22_gazebo_pos/meshes/alt_plaka.stl" scale="0.001 0.001 0.001"/>
-    </geometry>
-    <material name="silver"/>
-  </visual>
-  <collision>
-    <origin rpy="0 0 0" xyz="0 0 0"/>
-    <geometry>
-      <mesh filename="package://arm_22_gazebo_pos/meshes/alt_plaka.stl" scale="0.001 0.001 0.001"/>
-    </geometry>
-  </collision>
-</link>
-<link name="1_2_link_1">
-  <inertial>
-    <origin rpy="0 0 0" xyz="-4.440892098500626e-18 1.4354722485038024e-15 0.07105772806777622"/>
-    <mass value="4.533031384288756"/>
-    <inertia ixx="0.01043" ixy="-0.0" ixz="-0.0" iyy="0.007523" iyz="0.0" izz="0.004306"/>
-  </inertial>
-  <visual>
-    <origin rpy="0 0 0" xyz="-0.0 -0.0 -0.0535"/>
-    <geometry>
-      <mesh filename="package://arm_22_gazebo_pos/meshes/1_2_link_1.stl" scale="0.001 0.001 0.001"/>
-    </geometry>
-    <material name="silver"/>
-  </visual>
-  <collision>
-    <origin rpy="0 0 0" xyz="-0.0 -0.0 -0.0535"/>
-    <geometry>
-      <mesh filename="package://arm_22_gazebo_pos/meshes/1_2_link_1.stl" scale="0.001 0.001 0.001"/>
-    </geometry>
-  </collision>
-</link>
-<link name="2_3_link_1">
-  <inertial>
-    <origin rpy="0 0 0" xyz="-0.021499999999999762 1.9407189213085804e-17 0.40425517026841495"/>
-    <mass value="11.422793723409663"/>
-    <inertia ixx="0.493811" ixy="-0.0" ixz="-0.0" iyy="0.49327" iyz="-0.0" izz="0.005454"/>
-  </inertial>
-  <visual>
-    <origin rpy="0 0 0" xyz="-0.0215 -0.0 -0.141"/>
-    <geometry>
-      <mesh filename="package://arm_22_gazebo_pos/meshes/2_3_link_1.stl" scale="0.001 0.001 0.001"/>
-    </geometry>
-    <material name="silver"/>
-  </visual>
-  <collision>
-    <origin rpy="0 0 0" xyz="-0.0215 -0.0 -0.141"/>
-    <geometry>
-      <mesh filename="package://arm_22_gazebo_pos/meshes/2_3_link_1.stl" scale="0.001 0.001 0.001"/>
-    </geometry>
-  </collision>
-</link>
-<link name="3_4_link_1">
-  <inertial>
-    <origin rpy="0 0 0" xyz="0.025000000000004786 -0.11600699772151865 1.1102230246251565e-16"/>
-    <mass value="2.1095820437502777"/>
-    <inertia ixx="0.004579" ixy="0.0" ixz="0.0" iyy="0.003013" iyz="0.0" izz="0.005799"/>
-  </inertial>
-  <visual>
-    <origin rpy="0 0 0" xyz="0.025 -0.0 -0.7965"/>
-    <geometry>
-      <mesh filename="package://arm_22_gazebo_pos/meshes/3_4_link_1.stl" scale="0.001 0.001 0.001"/>
-    </geometry>
-    <material name="silver"/>
-  </visual>
-  <collision>
-    <origin rpy="0 0 0" xyz="0.025 -0.0 -0.7965"/>
-    <geometry>
-      <mesh filename="package://arm_22_gazebo_pos/meshes/3_4_link_1.stl" scale="0.001 0.001 0.001"/>
-    </geometry>
-  </collision>
-</link>
-<link name="4_5_link_1">
-  <inertial>
-    <origin rpy="0 0 0" xyz="0.02631095454187837 -0.25285048089107715 1.1102230246251565e-16"/>
-    <mass value="6.936333570954899"/>
-    <inertia ixx="0.111412" ixy="0.023035" ixz="0.0" iyy="0.014343" iyz="0.0" izz="0.122701"/>
-  </inertial>
-  <visual>
-    <origin rpy="0 0 0" xyz="-0.0 0.14925 -0.7965"/>
-    <geometry>
-      <mesh filename="package://arm_22_gazebo_pos/meshes/4_5_link_1.stl" scale="0.001 0.001 0.001"/>
-    </geometry>
-    <material name="silver"/>
-  </visual>
-  <collision>
-    <origin rpy="0 0 0" xyz="-0.0 0.14925 -0.7965"/>
-    <geometry>
-      <mesh filename="package://arm_22_gazebo_pos/meshes/4_5_link_1.stl" scale="0.001 0.001 0.001"/>
-    </geometry>
-  </collision>
-</link>
-<link name="5_6_link_1">
-  <inertial>
-    <origin rpy="0 0 0" xyz="-0.03519954944823235 0.0 1.1102230246251565e-16"/>
-    <mass value="1.380651703874357"/>
-    <inertia ixx="0.000555" ixy="0.0" ixz="0.0" iyy="0.00102" iyz="0.0" izz="0.000981"/>
-  </inertial>
-  <visual>
-    <origin rpy="0 0 0" xyz="-0.055 0.54725 -0.7965"/>
-    <geometry>
-      <mesh filename="package://arm_22_gazebo_pos/meshes/5_6_link_1.stl" scale="0.001 0.001 0.001"/>
-    </geometry>
-    <material name="silver"/>
-  </visual>
-  <collision>
-    <origin rpy="0 0 0" xyz="-0.055 0.54725 -0.7965"/>
-    <geometry>
-      <mesh filename="package://arm_22_gazebo_pos/meshes/5_6_link_1.stl" scale="0.001 0.001 0.001"/>
-    </geometry>
-  </collision>
-</link>
-<link name="gripper_link_1">
-  <inertial>
-    <origin rpy="0 0 0" xyz="-1.9022434799199985e-14 -0.03416319786748656 0.0010518735260454104"/>
-    <mass value="0.17794522906388674"/>
-    <inertia ixx="0.000124" ixy="-0.0" ixz="0.0" iyy="0.000145" iyz="-1e-06" izz="0.000206"/>
-  </inertial>
-  <visual>
-    <origin rpy="0 0 0" xyz="-0.0 0.56925 -0.7965"/>
-    <geometry>
-      <mesh filename="package://arm_22_gazebo_pos/meshes/gripper_link_1.stl" scale="0.001 0.001 0.001"/>
-    </geometry>
-    <material name="silver"/>
-  </visual>
-  <collision>
-    <origin rpy="0 0 0" xyz="-0.0 0.56925 -0.7965"/>
-    <geometry>
-      <mesh filename="package://arm_22_gazebo_pos/meshes/gripper_link_1.stl" scale="0.001 0.001 0.001"/>
-    </geometry>
-  </collision>
-</link>
-<link name="parmak_1_link_1">
-  <inertial>
-    <origin rpy="0 0 0" xyz="-0.001967084910946904 -0.04536035309441244 -0.010499999999999954"/>
-    <mass value="0.17651437470268025"/>
-    <inertia ixx="0.000124" ixy="-0.0" ixz="0.0" iyy="9e-06" iyz="0.0" izz="0.00012"/>
-  </inertial>
-  <visual>
-    <origin rpy="0 0 0" xyz="0.008 0.65425 -0.8115"/>
-    <geometry>
-      <mesh filename="package://arm_22_gazebo_pos/meshes/parmak_1_link_1.stl" scale="0.001 0.001 0.001"/>
-    </geometry>
-    <material name="silver"/>
-  </visual>
-  <collision>
-    <origin rpy="0 0 0" xyz="0.008 0.65425 -0.8115"/>
-    <geometry>
-      <mesh filename="package://arm_22_gazebo_pos/meshes/parmak_1_link_1.stl" scale="0.001 0.001 0.001"/>
-    </geometry>
-  </collision>
-</link>
-<link name="parmak_2_link_1">
-  <inertial>
-    <origin rpy="0 0 0" xyz="0.0019670849109472976 -0.045360353094412664 -0.010499999999999954"/>
-    <mass value="0.17651437470268025"/>
-    <inertia ixx="0.000124" ixy="0.0" ixz="0.0" iyy="9e-06" iyz="0.0" izz="0.00012"/>
-  </inertial>
-  <visual>
-    <origin rpy="0 0 0" xyz="-0.008 0.65425 -0.8115"/>
-    <geometry>
-      <mesh filename="package://arm_22_gazebo_pos/meshes/parmak_2_link_1.stl" scale="0.001 0.001 0.001"/>
-    </geometry>
-    <material name="silver"/>
-  </visual>
-  <collision>
-    <origin rpy="0 0 0" xyz="-0.008 0.65425 -0.8115"/>
-    <geometry>
-      <mesh filename="package://arm_22_gazebo_pos/meshes/parmak_2_link_1.stl" scale="0.001 0.001 0.001"/>
-    </geometry>
-  </collision>
-</link>
-<joint name="axis_1" type="continuous">
-  <origin rpy="0 0 0" xyz="0.0 0.0 0.0535"/>
-  <parent link="alt_plaka"/>
-  <child link="1_2_link_1"/>
-  <axis xyz="0.0 0.0 1.0"/>
-</joint>
-<joint name="axis_2" type="continuous">
-  <origin rpy="0 0 0" xyz="0.0215 0.0 0.0875"/>
-  <parent link="1_2_link_1"/>
-  <child link="2_3_link_1"/>
-  <axis xyz="-1.0 0.0 0.0"/>
-</joint>
-<joint name="axis_3" type="continuous">
-  <origin rpy="0 0 0" xyz="-0.0465 0.0 0.6555"/>
-  <parent link="2_3_link_1"/>
-  <child link="3_4_link_1"/>
-  <axis xyz="-1.0 0.0 0.0"/>
-</joint>
-<joint name="axis_4" type="continuous">
-  <origin rpy="0 0 0" xyz="0.025 -0.14925 0.0"/>
-  <parent link="3_4_link_1"/>
-  <child link="4_5_link_1"/>
-  <axis xyz="-0.0 1.0 -0.0"/>
-</joint>
-<joint name="axis_5" type="continuous">
-  <origin rpy="0 0 0" xyz="0.055 -0.398 0.0"/>
-  <parent link="4_5_link_1"/>
-  <child link="5_6_link_1"/>
-  <axis xyz="-1.0 0.0 0.0"/>
-</joint>
-<joint name="axis_6" type="continuous">
-  <origin rpy="0 0 0" xyz="-0.055 -0.022 0.0"/>
-  <parent link="5_6_link_1"/>
-  <child link="gripper_link_1"/>
-  <axis xyz="-0.0 -1.0 0.0"/>
-</joint>
-<joint name="axis_parmak_1" type="revolute">
-  <origin rpy="0 0 0" xyz="-0.008 -0.085 0.015"/>
-  <parent link="gripper_link_1"/>
-  <child link="parmak_1_link_1"/>
-  <axis xyz="0.0 0.0 1.0"/>
-  <limit
-  lower="-0.5"
-  upper="0.05"
-  effort="200"
-  velocity="20" />
-</joint>
-<joint name="axis_parmak_2" type="revolute">
-  <origin rpy="0 0 0" xyz="0.008 -0.085 0.015"/>
-  <parent link="gripper_link_1"/>
-  <child link="parmak_2_link_1"/>
-  <axis xyz="0.0 0.0 1.0"/>
-  <limit
-  lower="-0.05"
-  upper="0.5"
-  effort="200"
-  velocity="20" />
-</joint>
+<robot name="assembly"
+  xmlns:xacro="http://www.ros.org/wiki/xacro">
+  <!-- <xacro:include filename="$(find arm_22_gazebo_pos)/urdf/materials.xacro" /> -->
+  <xacro:include filename="$(find arm_22_gazebo_pos)/urdf/assembly.trans" />
+  <xacro:include filename="$(find arm_22_gazebo_pos)/urdf/assembly.gazebo" />
+  <xacro:include filename="$(find rover_22_description)/urdf/rover_22.xacro" />
+  <!-- <link name="world"> </link> -->
+  <joint name="dummy_joint" type="fixed">
+    <origin xyz="0.39 0.3 0.07" rpy="0 0 3.14"/>
+    <parent link="base_link"/>
+    <child link="alt_plaka"/>
+  </joint>
+  <link name="alt_plaka">
+    <inertial>
+      <origin rpy="0 0 0" xyz="2.111478230178841e-13 0.011682408428370204 0.005554773279956959"/>
+      <mass value="4.192131083267752"/>
+      <inertia ixx="0.007549" ixy="0.0" ixz="0.0" iyy="0.013998" iyz="0.000517" izz="0.018961"/>
+    </inertial>
+    <visual>
+      <origin rpy="0 0 0" xyz="0 0 0"/>
+      <geometry>
+        <mesh filename="package://arm_22_gazebo_pos/meshes/alt_plaka.stl" scale="0.001 0.001 0.001"/>
+      </geometry>
+      <material name="silver"/>
+    </visual>
+    <collision>
+      <origin rpy="0 0 0" xyz="0 0 0"/>
+      <geometry>
+        <mesh filename="package://arm_22_gazebo_pos/meshes/alt_plaka.stl" scale="0.001 0.001 0.001"/>
+      </geometry>
+    </collision>
+  </link>
+  <link name="1_2_link_1">
+    <inertial>
+      <origin rpy="0 0 0" xyz="-4.440892098500626e-18 1.4354722485038024e-15 0.07105772806777622"/>
+      <mass value="4.533031384288756"/>
+      <inertia ixx="0.01043" ixy="-0.0" ixz="-0.0" iyy="0.007523" iyz="0.0" izz="0.004306"/>
+    </inertial>
+    <visual>
+      <origin rpy="0 0 0" xyz="-0.0 -0.0 -0.0535"/>
+      <geometry>
+        <mesh filename="package://arm_22_gazebo_pos/meshes/1_2_link_1.stl" scale="0.001 0.001 0.001"/>
+      </geometry>
+      <material name="silver"/>
+    </visual>
+    <collision>
+      <origin rpy="0 0 0" xyz="-0.0 -0.0 -0.0535"/>
+      <geometry>
+        <mesh filename="package://arm_22_gazebo_pos/meshes/1_2_link_1.stl" scale="0.001 0.001 0.001"/>
+      </geometry>
+    </collision>
+  </link>
+  <link name="2_3_link_1">
+    <inertial>
+      <origin rpy="0 0 0" xyz="-0.021499999999999762 1.9407189213085804e-17 0.40425517026841495"/>
+      <mass value="11.422793723409663"/>
+      <inertia ixx="0.493811" ixy="-0.0" ixz="-0.0" iyy="0.49327" iyz="-0.0" izz="0.005454"/>
+    </inertial>
+    <visual>
+      <origin rpy="0 0 0" xyz="-0.0215 -0.0 -0.141"/>
+      <geometry>
+        <mesh filename="package://arm_22_gazebo_pos/meshes/2_3_link_1.stl" scale="0.001 0.001 0.001"/>
+      </geometry>
+      <material name="silver"/>
+    </visual>
+    <collision>
+      <origin rpy="0 0 0" xyz="-0.0215 -0.0 -0.141"/>
+      <geometry>
+        <mesh filename="package://arm_22_gazebo_pos/meshes/2_3_link_1.stl" scale="0.001 0.001 0.001"/>
+      </geometry>
+    </collision>
+  </link>
+  <link name="3_4_link_1">
+    <inertial>
+      <origin rpy="0 0 0" xyz="0.025000000000004786 -0.11600699772151865 1.1102230246251565e-16"/>
+      <mass value="2.1095820437502777"/>
+      <inertia ixx="0.004579" ixy="0.0" ixz="0.0" iyy="0.003013" iyz="0.0" izz="0.005799"/>
+    </inertial>
+    <visual>
+      <origin rpy="0 0 0" xyz="0.025 -0.0 -0.7965"/>
+      <geometry>
+        <mesh filename="package://arm_22_gazebo_pos/meshes/3_4_link_1.stl" scale="0.001 0.001 0.001"/>
+      </geometry>
+      <material name="silver"/>
+    </visual>
+    <collision>
+      <origin rpy="0 0 0" xyz="0.025 -0.0 -0.7965"/>
+      <geometry>
+        <mesh filename="package://arm_22_gazebo_pos/meshes/3_4_link_1.stl" scale="0.001 0.001 0.001"/>
+      </geometry>
+    </collision>
+  </link>
+  <link name="4_5_link_1">
+    <inertial>
+      <origin rpy="0 0 0" xyz="0.02631095454187837 -0.25285048089107715 1.1102230246251565e-16"/>
+      <mass value="6.936333570954899"/>
+      <inertia ixx="0.111412" ixy="0.023035" ixz="0.0" iyy="0.014343" iyz="0.0" izz="0.122701"/>
+    </inertial>
+    <visual>
+      <origin rpy="0 0 0" xyz="-0.0 0.14925 -0.7965"/>
+      <geometry>
+        <mesh filename="package://arm_22_gazebo_pos/meshes/4_5_link_1.stl" scale="0.001 0.001 0.001"/>
+      </geometry>
+      <material name="silver"/>
+    </visual>
+    <collision>
+      <origin rpy="0 0 0" xyz="-0.0 0.14925 -0.7965"/>
+      <geometry>
+        <mesh filename="package://arm_22_gazebo_pos/meshes/4_5_link_1.stl" scale="0.001 0.001 0.001"/>
+      </geometry>
+    </collision>
+  </link>
+  <link name="5_6_link_1">
+    <inertial>
+      <origin rpy="0 0 0" xyz="-0.03519954944823235 0.0 1.1102230246251565e-16"/>
+      <mass value="1.380651703874357"/>
+      <inertia ixx="0.000555" ixy="0.0" ixz="0.0" iyy="0.00102" iyz="0.0" izz="0.000981"/>
+    </inertial>
+    <visual>
+      <origin rpy="0 0 0" xyz="-0.055 0.54725 -0.7965"/>
+      <geometry>
+        <mesh filename="package://arm_22_gazebo_pos/meshes/5_6_link_1.stl" scale="0.001 0.001 0.001"/>
+      </geometry>
+      <material name="silver"/>
+    </visual>
+    <collision>
+      <origin rpy="0 0 0" xyz="-0.055 0.54725 -0.7965"/>
+      <geometry>
+        <mesh filename="package://arm_22_gazebo_pos/meshes/5_6_link_1.stl" scale="0.001 0.001 0.001"/>
+      </geometry>
+    </collision>
+  </link>
+  <link name="gripper_link_1">
+    <inertial>
+      <origin rpy="0 0 0" xyz="-1.9022434799199985e-14 -0.03416319786748656 0.0010518735260454104"/>
+      <mass value="0.17794522906388674"/>
+      <inertia ixx="0.000124" ixy="-0.0" ixz="0.0" iyy="0.000145" iyz="-1e-06" izz="0.000206"/>
+    </inertial>
+    <visual>
+      <origin rpy="0 0 0" xyz="-0.0 0.56925 -0.7965"/>
+      <geometry>
+        <mesh filename="package://arm_22_gazebo_pos/meshes/gripper_link_1.stl" scale="0.001 0.001 0.001"/>
+      </geometry>
+      <material name="silver"/>
+    </visual>
+    <collision>
+      <origin rpy="0 0 0" xyz="-0.0 0.56925 -0.7965"/>
+      <geometry>
+        <mesh filename="package://arm_22_gazebo_pos/meshes/gripper_link_1.stl" scale="0.001 0.001 0.001"/>
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